File: Hardware/PCB/KiCad6/ESP32_programmer.kicad_sch (KiCad schematic)
At the start: 20 parts, among them J9 USB_B_Micro, Q5 BC817, Q6 BC817, SW1 PROG, SW2 RST, U3 AZ1117-3.3, U4 CH340C

Commit message: PCB Update from current schema
Parts:
- renumbered C15 to C16, C16 to C17, C17 to C18
Changed lines of the file:
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@@
   (symbol (lib_id "power:+3.3V") (at 96.52 26.67 0) (unit 1)
     (in_bom yes) (on_board yes) (fields_autoplaced)
-    (property "Reference" "#PWR057" (id 0) (at 96.52 30.48 0)
+    (property "Reference" "#PWR061" (id 0) (at 96.52 30.48 0)
       (effects (font (size 1.27 1.27)) hide)
     )
@@
   (symbol (lib_id "power:GND") (at 93.98 67.31 0) (unit 1)
     (in_bom yes) (on_board yes) (fields_autoplaced)
-    (property "Reference" "#PWR056" (id 0) (at 93.98 73.66 0)
+    (property "Reference" "#PWR060" (id 0) (at 93.98 73.66 0)
       (effects (font (size 1.27 1.27)) hide)
     )
@@
   (symbol (lib_id "power:GND") (at 105.41 110.49 0) (unit 1)
     (in_bom yes) (on_board yes) (fields_autoplaced)
-    (property "Reference" "#PWR060" (id 0) (at 105.41 116.84 0)
+    (property "Reference" "#PWR064" (id 0) (at 105.41 116.84 0)
       (effects (font (size 1.27 1.27)) hide)
     )
@@
   (symbol (lib_id "power:+5V") (at 68.58 64.77 0) (unit 1)
     (in_bom yes) (on_board yes) (fields_autoplaced)
-    (property "Reference" "#PWR054" (id 0) (at 68.58 68.58 0)
+    (property "Reference" "#PWR058" (id 0) (at 68.58 68.58 0)
       (effects (font (size 1.27 1.27)) hide)
     )
@@
   (symbol (lib_id "power:GND") (at 187.96 40.64 0) (unit 1)
     (in_bom yes) (on_board yes) (fields_autoplaced)
-    (property "Reference" "#PWR063" (id 0) (at 187.96 46.99 0)
+    (property "Reference" "#PWR067" (id 0) (at 187.96 46.99 0)
       (effects (font (size 1.27 1.27)) hide)
     )
@@
   (symbol (lib_id "power:GND") (at 215.9 74.93 0) (unit 1)
     (in_bom yes) (on_board yes) (fields_autoplaced)
-    (property "Reference" "#PWR064" (id 0) (at 215.9 81.28 0)
+    (property "Reference" "#PWR068" (id 0) (at 215.9 81.28 0)
       (effects (font (size 1.27 1.27)) hide)
     )
@@
   (symbol (lib_id "Device:C") (at 99.06 66.04 90) (unit 1)
     (in_bom yes) (on_board yes) (fields_autoplaced)
-    (property "Reference" "C17" (id 0) (at 99.06 58.42 90))
+    (property "Reference" "C18" (id 0) (at 99.06 58.42 90))
     (property "Value" "100nF" (id 1) (at 99.06 60.96 90))
     (property "Footprint" "Capacitor_SMD:C_0805_2012Metric_Pad1.18x1.45mm_HandSolder" (id 2) (at 102.87 65.0748 0)
@@
   (symbol (lib_id "power:+3.3V") (at 186.69 106.68 0) (unit 1)
     (in_bom yes) (on_board yes) (fields_autoplaced)
-    (property "Reference" "#PWR062" (id 0) (at 186.69 110.49 0)
+    (property "Reference" "#PWR066" (id 0) (at 186.69 110.49 0)
       (effects (font (size 1.27 1.27)) hide)
     )
@@
   (symbol (lib_id "power:GND") (at 215.9 92.71 0) (unit 1)
     (in_bom yes) (on_board yes) (fields_autoplaced)
-    (property "Reference" "#PWR065" (id 0) (at 215.9 99.06 0)
+    (property "Reference" "#PWR069" (id 0) (at 215.9 99.06 0)
       (effects (font (size 1.27 1.27)) hide)
     )
@@
   (symbol (lib_id "power:GND") (at 251.46 40.64 0) (unit 1)
     (in_bom yes) (on_board yes) (fields_autoplaced)
-    (property "Reference" "#PWR067" (id 0) (at 251.46 46.99 0)
+    (property "Reference" "#PWR071" (id 0) (at 251.46 46.99 0)
       (effects (font (size 1.27 1.27)) hide)
     )
@@
   (symbol (lib_id "power:GND") (at 215.9 111.76 0) (unit 1)
     (in_bom yes) (on_board yes) (fields_autoplaced)
-    (property "Reference" "#PWR066" (id 0) (at 215.9 118.11 0)
+    (property "Reference" "#PWR070" (id 0) (at 215.9 118.11 0)
       (effects (font (size 1.27 1.27)) hide)
     )
@@
   (symbol (lib_id "Device:C") (at 96.52 39.37 180) (unit 1)
     (in_bom yes) (on_board yes) (fields_autoplaced)
-    (property "Reference" "C16" (id 0) (at 100.33 38.0999 0)
+    (property "Reference" "C17" (id 0) (at 100.33 38.0999 0)
       (effects (font (size 1.27 1.27)) (justify right))
     )
@@
   (symbol (lib_id "power:GND") (at 81.28 44.45 0) (unit 1)
     (in_bom yes) (on_board yes) (fields_autoplaced)
-    (property "Reference" "#PWR055" (id 0) (at 81.28 50.8 0)
+    (property "Reference" "#PWR059" (id 0) (at 81.28 50.8 0)
       (effects (font (size 1.27 1.27)) hide)
     )
@@
   (symbol (lib_id "power:GND") (at 60.96 104.14 0) (unit 1)
     (in_bom yes) (on_board yes) (fields_autoplaced)
-    (property "Reference" "#PWR053" (id 0) (at 60.96 110.49 0)
+    (property "Reference" "#PWR057" (id 0) (at 60.96 110.49 0)
       (effects (font (size 1.27 1.27)) hide)
     )
@@
   (symbol (lib_id "power:+5V") (at 186.69 87.63 0) (unit 1)
     (in_bom yes) (on_board yes) (fields_autoplaced)
-    (property "Reference" "#PWR061" (id 0) (at 186.69 91.44 0)
+    (property "Reference" "#PWR065" (id 0) (at 186.69 91.44 0)
       (effects (font (size 1.27 1.27)) hide)
     )
@@
   (symbol (lib_id "power:GND") (at 96.52 45.72 0) (unit 1)
     (in_bom yes) (on_board yes) (fields_autoplaced)
-    (property "Reference" "#PWR058" (id 0) (at 96.52 52.07 0)
+    (property "Reference" "#PWR062" (id 0) (at 96.52 52.07 0)
       (effects (font (size 1.27 1.27)) hide)
     )
@@
   (symbol (lib_id "power:+3.3V") (at 105.41 62.23 0) (unit 1)
     (in_bom yes) (on_board yes) (fields_autoplaced)
-    (property "Reference" "#PWR059" (id 0) (at 105.41 66.04 0)
+    (property "Reference" "#PWR063" (id 0) (at 105.41 66.04 0)
       (effects (font (size 1.27 1.27)) hide)
     )
@@
   (symbol (lib_id "power:GND") (at 46.99 69.85 0) (unit 1)
     (in_bom yes) (on_board yes) (fields_autoplaced)
-    (property "Reference" "#PWR052" (id 0) (at 46.99 76.2 0)
+    (property "Reference" "#PWR056" (id 0) (at 46.99 76.2 0)
       (effects (font (size 1.27 1.27)) hide)
     )
@@
   (symbol (lib_id "Device:C") (at 54.61 67.31 90) (unit 1)
     (in_bom yes) (on_board yes) (fields_autoplaced)
-    (property "Reference" "C15" (id 0) (at 54.61 59.69 90))
+    (property "Reference" "C16" (id 0) (at 54.61 59.69 90))
     (property "Value" "4.7uF" (id 1) (at 54.61 62.23 90))
     (property "Footprint" "Capacitor_SMD:C_0805_2012Metric_Pad1.18x1.45mm_HandSolder" (id 2) (at 58.42 66.3448 0)
